File: pcb/tt08_cw_keyer.kicad_pcb (KiCad board)
At the start: 2 copper layers, 20.3 x 46.2 mm, 26 parts, among them J1 ASJ-200-B-HT, J2 ASJ-200-B-HT, J3 Conn_02x06_PMOD, Q1 MBT3904DW1, Q2 MBT3904DW1, Q3 MBT3904DW1, SW1 TS11-674-55-BK-100-RA-D, SW2 TS11-674-55-BK-100-RA-D

Commit message: Update PCB to correct DRC errors, unconventional audio jack pads, edge clearance
Parts:
- moved Q2 0.25 mm to (117.0, 90.2)
- moved J2 0.20 mm to (116.0, 90.2)
Routing:
- net GND: track 11.8 -> 21.3 mm, vias 4 -> 7
- net Net-(Q2B-B2): track 50.2 -> 47.4 mm
